File: FG_Controller/older_versions/V0.4/FG_Controller.kicad_pcb (KiCad board)
At the start: 2 copper layers, 220 x 130 mm, 70 parts, among them J1 USB_C_Receptacle_USB2.0_16P, J2 JST- 1.00mm 4 Pin, SW1 SW_Push, SW2 SW_Push, U1 RP2040, U2 USBLC6-2SC6, U3 AP2127N3-1.2, U4 W25Q16JVSS, U5 ER_OLEDM0.91_1x-I2C, Y1 12MHz Crystal 3225

Commit message: Update PCB 0.5 + Casing step files
Parts:
- H1, H2, H3, H4, H5: footprint MountingHole:MountingHole_3.2mm_M3_DIN965_Pad_TopBottom -> MountingHole:MountingHole_3.2mm_M3_DIN965_Pad_TopOnly
- SW1, SW2: moved to B.Cu
- moved U5 197.7 mm to (255.2, 56.0)
- moved C17 172.6 mm to (242.8, 32.0), turned to 0 degrees
- moved SW1 114.0 mm to (25.0, 37.9), turned to 180 degrees
- moved C4 111.0 mm to (24.7, 32.0)
- moved C6 97.9 mm to (22.8, 45.5)
- moved SW2 92.6 mm to (25.0, 56.5), turned to 180 degrees
- moved Start1 34.4 mm to (267.5, 21.5)
- moved H3 31.0 mm to (275.0, 16.0)
- moved H4 31.0 mm to (275.0, 135.0)
- moved Select1 28.4 mm to (248.5, 21.5)
- moved H1 21.0 mm to (15.0, 16.0)
- moved H2 21.0 mm to (15.0, 135.0)
- moved Humanity is way more interesting than any miracle 15.3 mm to (37.5, 101.5)
Routing:
- net GND: track 390.4 -> 517.2 mm, vias 21 -> 29
- net +3V3: track 261.7 -> 377.6 mm, vias 12 -> 15
- net /CS_: track 48.7 -> 162.9 mm, vias 2 -> 3
- net /RUN_: track 66.1 -> 165.0 mm, vias 2 -> 3
- net GP25: track 179.6 -> 87.3 mm
- net GP24: track 172.8 -> 88.2 mm, vias 1 -> 0
- net GP17: track 303.8 -> 351.2 mm
- net GP10: track 79.9 -> 113.5 mm
- net GP26: track 54.4 -> 82.0 mm
- net GP18: track 274.6 -> 270.2 mm
- removed copper zone on B.Cu, net GND
Other:
- board size 220 x 130 mm -> 270 x 129 mm
- board text added: "Pearl V0.4"
- board text removed: "Pearl V0.5"
